Commit message: preparing for submission

File: urdf/my_robot.xacro (robot description, xacro)
@@ -209,5 +209,5 @@
   </link>
   <joint name="camera_joint" type="fixed">
-    <origin xyz="0.12 0.0 0.05" rpy="0.0 0.0 0.0"/>
+    <origin xyz="0.15 0.0 0.05" rpy="0.0 0.0 0.0"/>
     <parent link="chassis"/>
     <child link="camera"/>
@@ -236,4 +236,11 @@
       </geometry>
     </collision>
+  </link>
+  <joint name="camera_optical_joint" type="fixed">
+    <origin xyz="0.0 0.0 0.0" rpy="-1.5707 0.0 -1.5707"/>
+    <parent link="camera"/>
+    <child link="camera_link_optical"/>
+  </joint>
+  <link name="camera_link_optical">
   </link>
   <joint name="hokuyo_joint" type="fixed">
